File: ai03-pcb-guide.kicad_pcb (KiCad board)
At the start: 2 copper layers, 76.2 x 38.1 mm, 24 parts, among them SW1 SW_Push, U1 ATmega32U4-AU, Y1 Crystal_GND24_Small

Commit message: lmao wtf
Parts:
- removed F1: 500mA, Fuse_Holders_and_Fuses:Fuse_SMD1206_Reflow
- removed SW1: SW_Push, random-keyboard-parts:SKQG-1155865
- added D10: SOD-123, Diode_SMD:D_0805_2012Metric, F.Cu at (66.6, 18.4)
- added D11: SOD-123, Diode_SMD:D_0805_2012Metric, F.Cu at (66.6, 15.3)
- added D12: SOD-123, Diode_SMD:D_0805_2012Metric, F.Cu at (71.0, 21.4)
- added D13: SOD-123, Diode_SMD:D_0805_2012Metric, F.Cu at (64.8, 28.7)
- added D14: SOD-123, Diode_SMD:D_0805_2012Metric, F.Cu at (75.5, 18.4)
- added D15: SOD-123, Diode_SMD:D_0805_2012Metric, F.Cu at (70.1, 24.4)
- added D16: SOD-123, Diode_SMD:D_0805_2012Metric, F.Cu at (79.9, 15.3)
- added D17: SOD-123, Diode_SMD:D_0805_2012Metric, F.Cu at (60.4, 36.1)
- added D18: SOD-123, Diode_SMD:D_0805_2012Metric, F.Cu at (64.8, 31.7)
- added D19: SOD-123, Diode_SMD:D_0805_2012Metric, F.Cu at (70.1, 27.5)
- added D20: SOD-123, Diode_SMD:D_0805_2012Metric, F.Cu at (75.5, 21.4)
- added D21: SOD-123, Diode_SMD:D_0805_2012Metric, F.Cu at (79.9, 18.4)
- added D22: SOD-123, Diode_SMD:D_0805_2012Metric, F.Cu at (74.5, 24.4)
- added D23: SOD-123, Diode_SMD:D_0805_2012Metric, F.Cu at (84.4, 15.3)
- added D24: SOD-123, Diode_SMD:D_0805_2012Metric, F.Cu at (60.4, 33.1)
- added D25: SOD-123, Diode_SMD:D_0805_2012Metric, F.Cu at (74.5, 27.5)
- added D26: SOD-123, Diode_SMD:D_0805_2012Metric, F.Cu at (78.2, 30.5)
- added D27: SOD-123, Diode_SMD:D_0805_2012Metric, F.Cu at (93.3, 15.3)
- added D28: SOD-123, Diode_SMD:D_0805_2012Metric, F.Cu at (73.7, 33.6)
- added D29: SOD-123, Diode_SMD:D_0805_2012Metric, F.Cu at (83.4, 24.4)
- added D30: SOD-123, Diode_SMD:D_0805_2012Metric, F.Cu at (88.8, 18.4)
- added D31: SOD-123, Diode_SMD:D_0805_2012Metric, F.Cu at (84.4, 21.4)
- added D32: SOD-123, Diode_SMD:D_0805_2012Metric, F.Cu at (69.3, 36.6)
- added D33: SOD-123, Diode_SMD:D_0805_2012Metric, F.Cu at (69.3, 30.5)
- added D34: SOD-123, Diode_SMD:D_0805_2012Metric, F.Cu at (73.7, 30.5)
- added D35: SOD-123, Diode_SMD:D_0805_2012Metric, F.Cu at (88.8, 15.3)
- added D36: SOD-123, Diode_SMD:D_0805_2012Metric, F.Cu at (69.3, 33.6)
- added D37: SOD-123, Diode_SMD:D_0805_2012Metric, F.Cu at (79.0, 24.4)
- added D38: SOD-123, Diode_SMD:D_0805_2012Metric, F.Cu at (64.8, 37.8)
- added D39: SOD-123, Diode_SMD:D_0805_2012Metric, F.Cu at (84.4, 18.4)
- added D40: SOD-123, Diode_SMD:D_0805_2012Metric, F.Cu at (79.9, 21.4)
- added D41: SOD-123, Diode_SMD:D_0805_2012Metric, F.Cu at (64.8, 34.7)
- added D42: SOD-123, Diode_SMD:D_0805_2012Metric, F.Cu at (79.0, 27.5)
- added D43: SOD-123, Diode_SMD:D_0805_2012Metric, F.Cu at (83.4, 27.5)
- added D44: SOD-123, Diode_SMD:D_0805_2012Metric, F.Cu at (93.3, 21.4)
- added D45: SOD-123, Diode_SMD:D_0805_2012Metric, F.Cu at (78.2, 36.6)
- added D46: SOD-123, Diode_SMD:D_0805_2012Metric, F.Cu at (87.9, 27.5)
- added D47: SOD-123, Diode_SMD:D_0805_2012Metric, F.Cu at (82.6, 30.5)
- added D48: SOD-123, Diode_SMD:D_0805_2012Metric, F.Cu at (78.2, 33.6)
- added D49: SOD-123, Diode_SMD:D_0805_2012Metric, F.Cu at (87.9, 24.4)
- added D5: SOD-123, Diode_SMD:D_0805_2012Metric, F.Cu at (60.4, 30.1)
- added D50: SOD-123, Diode_SMD:D_0805_2012Metric, F.Cu at (93.3, 18.4)
- added D51: SOD-123, Diode_SMD:D_0805_2012Metric, F.Cu at (88.8, 21.4)
- added D52: SOD-123, Diode_SMD:D_0805_2012Metric, F.Cu at (73.7, 36.6)
- added D53: SOD-123, Diode_SMD:D_0805_2012Metric, F.Cu at (92.3, 24.4)
- added D54: SOD-123, Diode_SMD:D_0805_2012Metric, F.Cu at (55.9, 30.1)
- added D6: SOD-123, Diode_SMD:D_0805_2012Metric, F.Cu at (71.0, 18.4)
- added D7: SOD-123, Diode_SMD:D_0805_2012Metric, F.Cu at (65.6, 25.6)
- added D8: SOD-123, Diode_SMD:D_0805_2012Metric, F.Cu at (75.5, 15.3)
- added D9: SOD-123, Diode_SMD:D_0805_2012Metric, F.Cu at (55.9, 36.1)
- added MX10: MX-NoLED-MX_Alps_Hybrid, gHeavyIndustries:MX-Alps-Choc-X-1U-NoLED, F.Cu at (-93.3, 20.6)
- added MX11: MX-NoLED-MX_Alps_Hybrid, gHeavyIndustries:MX-Alps-Choc-X-1U-NoLED, F.Cu at (-73.1, 0.35)
- added MX12: MX-NoLED-MX_Alps_Hybrid, gHeavyIndustries:MX-Alps-Choc-X-1U-NoLED, F.Cu at (-52.9, -19.8)
- added MX13: MX-NoLED-MX_Alps_Hybrid, gHeavyIndustries:MX-Alps-Choc-X-1U-NoLED, F.Cu at (-160.0, -6.35)
- added MX14: MX-NoLED-MX_Alps_Hybrid, gHeavyIndustries:MX-Alps-Choc-X-1U-NoLED, F.Cu at (-160.0, 12.7)
- added MX15: MX-NoLED-MX_Alps_Hybrid, gHeavyIndustries:MX-Alps-Choc-X-1U-NoLED, F.Cu at (-93.3, -40.0)
- added MX16: MX-NoLED-MX_Alps_Hybrid, gHeavyIndustries:MX-Alps-Choc-X-1U-NoLED, F.Cu at (-73.1, 20.6)
- added MX17: MX-NoLED-MX_Alps_Hybrid, gHeavyIndustries:MX-Alps-Choc-X-1U-NoLED, F.Cu at (-52.9, 0.35)
- added MX18: MX-NoLED-MX_Alps_Hybrid, gHeavyIndustries:MX-Alps-Choc-X-1U-NoLED, F.Cu at (-32.7, -19.8)
- added MX19: MX-NoLED-MX_Alps_Hybrid, gHeavyIndustries:MX-Alps-Choc-X-1U-NoLED, F.Cu at (-12.5, -40.0)
- added MX20: MX-NoLED-MX_Alps_Hybrid, gHeavyIndustries:MX-Alps-Choc-X-1U-NoLED, F.Cu at (7.73, -60.2)
- added MX21: MX-NoLED-MX_Alps_Hybrid, gHeavyIndustries:MX-Alps-Choc-X-1U-NoLED, F.Cu at (-73.1, 40.8)
- added MX22: MX-NoLED-MX_Alps_Hybrid, gHeavyIndustries:MX-Alps-Choc-X-1U-NoLED, F.Cu at (-52.9, 20.6)
- added MX23: MX-NoLED-MX_Alps_Hybrid, gHeavyIndustries:MX-Alps-Choc-X-1U-NoLED, F.Cu at (-32.7, 0.35)
- added MX24: MX-NoLED-MX_Alps_Hybrid, gHeavyIndustries:MX-Alps-Choc-X-1U-NoLED, F.Cu at (-12.5, -19.8)
- added MX25: MX-NoLED-MX_Alps_Hybrid, gHeavyIndustries:MX-Alps-Choc-X-1U-NoLED, F.Cu at (7.73, -40.0)
- added MX26: MX-NoLED-MX_Alps_Hybrid, gHeavyIndustries:MX-Alps-Choc-X-1U-NoLED, F.Cu at (27.9, -60.2)
- added MX27: MX-NoLED-MX_Alps_Hybrid, gHeavyIndustries:MX-Alps-Choc-X-1U-NoLED, F.Cu at (-52.9, 40.8)
- added MX28: MX-NoLED-MX_Alps_Hybrid, gHeavyIndustries:MX-Alps-Choc-X-1U-NoLED, F.Cu at (-32.7, 20.6)
- added MX29: MX-NoLED-MX_Alps_Hybrid, gHeavyIndustries:MX-Alps-Choc-X-1U-NoLED, F.Cu at (-12.5, -60.2)
- added MX30: MX-NoLED-MX_Alps_Hybrid, gHeavyIndustries:MX-Alps-Choc-X-1U-NoLED, F.Cu at (7.73, -19.8)
- added MX31: MX-NoLED-MX_Alps_Hybrid, gHeavyIndustries:MX-Alps-Choc-X-1U-NoLED, F.Cu at (-160.0, -25.4)
- added MX32: MX-NoLED-MX_Alps_Hybrid, gHeavyIndustries:MX-Alps-Choc-X-1U-NoLED, F.Cu at (-141.0, -6.35)
- added MX33: MX-NoLED-MX_Alps_Hybrid, gHeavyIndustries:MX-Alps-Choc-X-1U-NoLED, F.Cu at (-32.7, 40.8)
- added MX34: MX-NoLED-MX_Alps_Hybrid, gHeavyIndustries:MX-Alps-Choc-X-1U-NoLED, F.Cu at (-12.5, 20.6)
- added MX35: MX-NoLED-MX_Alps_Hybrid, gHeavyIndustries:MX-Alps-Choc-X-1U-NoLED, F.Cu at (7.73, 0.35)
- added MX36: MX-NoLED-MX_Alps_Hybrid, gHeavyIndustries:MX-Alps-Choc-X-1U-NoLED, F.Cu at (27.9, -19.8)
- added MX37: MX-NoLED-MX_Alps_Hybrid, gHeavyIndustries:MX-Alps-Choc-X-1U-NoLED, F.Cu at (48.1, -40.0)
- added MX38: MX-NoLED-MX_Alps_Hybrid, gHeavyIndustries:MX-Alps-Choc-X-1U-NoLED, F.Cu at (68.3, -60.2)
- added MX39: MX-NoLED-MX_Alps_Hybrid, gHeavyIndustries:MX-Alps-Choc-X-1U-NoLED, F.Cu at (-12.5, 40.8)
- added MX40: MX-NoLED-MX_Alps_Hybrid, gHeavyIndustries:MX-Alps-Choc-X-1U-NoLED, F.Cu at (7.73, 20.6)
- added MX41: MX-NoLED-MX_Alps_Hybrid, gHeavyIndustries:MX-Alps-Choc-X-1U-NoLED, F.Cu at (27.9, 0.35)
- added MX42: MX-NoLED-MX_Alps_Hybrid, gHeavyIndustries:MX-Alps-Choc-X-1U-NoLED, F.Cu at (-12.5, 0.35)
- added MX43: MX-NoLED-MX_Alps_Hybrid, gHeavyIndustries:MX-Alps-Choc-X-1U-NoLED, F.Cu at (48.1, -19.8)
- added MX44: MX-NoLED-MX_Alps_Hybrid, gHeavyIndustries:MX-Alps-Choc-X-1U-NoLED, F.Cu at (68.3, -40.0)
- added MX45: MX-NoLED-MX_Alps_Hybrid, gHeavyIndustries:MX-Alps-Choc-X-1U-NoLED, F.Cu at (88.5, -60.2)
- added MX46: MX-NoLED-MX_Alps_Hybrid, gHeavyIndustries:MX-Alps-Choc-X-1U-NoLED, F.Cu at (7.73, 40.8)
- added MX47: MX-NoLED-MX_Alps_Hybrid, gHeavyIndustries:MX-Alps-Choc-X-1U-NoLED, F.Cu at (27.9, 20.6)
- added MX48: MX-NoLED-MX_Alps_Hybrid, gHeavyIndustries:MX-Alps-Choc-X-1U-NoLED, F.Cu at (48.1, 0.35)
- added MX49: MX-NoLED-MX_Alps_Hybrid, gHeavyIndustries:MX-Alps-Choc-X-1U-NoLED, F.Cu at (68.3, -19.8)
- added MX5: MX-NoLED-MX_Alps_Hybrid, gHeavyIndustries:MX-Alps-Choc-X-1U-NoLED, F.Cu at (-52.9, -60.2)
- added MX50: MX-NoLED-MX_Alps_Hybrid, gHeavyIndustries:MX-Alps-Choc-X-1U-NoLED, F.Cu at (88.5, -40.0)
- added MX51: MX-NoLED-MX_Alps_Hybrid, gHeavyIndustries:MX-Alps-Choc-X-1U-NoLED, F.Cu at (27.9, 40.8)
- added MX52: MX-NoLED-MX_Alps_Hybrid, gHeavyIndustries:MX-Alps-Choc-X-1U-NoLED, F.Cu at (48.1, 20.6)
- added MX53: MX-NoLED-MX_Alps_Hybrid, gHeavyIndustries:MX-Alps-Choc-X-1U-NoLED, F.Cu at (68.3, 0.35)
- added MX54: MX-NoLED-MX_Alps_Hybrid, gHeavyIndustries:MX-Alps-Choc-X-1U-NoLED, F.Cu at (88.5, -19.8)
- added MX6: MX-NoLED-MX_Alps_Hybrid, gHeavyIndustries:MX-Alps-Choc-X-1U-NoLED, F.Cu at (-93.3, 0.35)
- added MX7: MX-NoLED-MX_Alps_Hybrid, gHeavyIndustries:MX-Alps-Choc-X-1U-NoLED, F.Cu at (-73.1, -19.8)
- added MX8: MX-NoLED-MX_Alps_Hybrid, gHeavyIndustries:MX-Alps-Choc-X-1U-NoLED, F.Cu at (-52.9, -40.0)
- added MX9: MX-NoLED-MX_Alps_Hybrid, gHeavyIndustries:MX-Alps-Choc-X-1U-NoLED, F.Cu at (-32.7, -60.2)
- C1, C2, C3, C4, C5, C6: footprint Capacitors_SMD:C_0805 -> Capacitor_SMD:C_0805_2012Metric; moved to F.Cu
- C7: value 10uF -> 0.1uF; footprint Capacitors_SMD:C_0805 -> Capacitor_SMD:C_0805_2012Metric; moved to F.Cu
- D1, D2, D3, D4: footprint Diodes_SMD:D_SOD-123 -> Diode_SMD:D_0805_2012Metric; moved to F.Cu
- MX1, MX2, MX3, MX4: value MX-NoLED -> MX-NoLED-MX_Alps_Hybrid; footprint MX_Alps_Hybrid:MX-1U -> gHeavyIndustries:MX-Alps-Choc-X-1U-NoLED
- R1, R2, R3, R4: footprint Resistors_SMD:R_0805 -> Resistor_SMD:R_0805_2012Metric; moved to F.Cu
- U1: footprint Housings_QFP:TQFP-44_10x10mm_Pitch0.8mm -> Package_QFP:TQFP-44_10x10mm_P0.8mm; moved to F.Cu
- USB1: footprint random-keyboard-parts:Molex-0548190589-Assembly -> random-keyboard-parts:Molex-0548190589; moved to F.Cu
- Y1: footprint Crystals:Crystal_SMD_3225-4pin_3.2x2.5mm -> Crystal:Crystal_SMD_3225-4Pin_3.2x2.5mm; moved to F.Cu
- moved MX2 216.2 mm to (-73.1, -60.2)
- moved MX4 215.5 mm to (-73.1, -40.0)
- moved MX3 204.9 mm to (-93.3, -19.8)
- moved MX1 175.4 mm to (-93.3, 40.8)
- moved R3 174.1 mm to (139.5, -67.3), turned to 0 degrees
- moved R4 159.6 mm to (49.3, -71.0), turned to 0 degrees
- moved U1 152.2 mm to (116.8, -58.4)
- moved R1 148.0 mm to (44.9, -74.0), turned to 0 degrees
- moved R2 145.0 mm to (44.9, -71.0), turned to 0 degrees
- moved D4 79.7 mm to (66.6, 21.4), turned to 0 degrees
- moved C3 74.8 mm to (96.7, 24.4), turned to 0 degrees
- moved D2 66.3 mm to (71.0, 15.3), turned to 0 degrees
- moved D3 65.4 mm to (55.9, 33.1), turned to 0 degrees
- moved C6 65.3 mm to (87.0, 30.5), turned to 0 degrees
- moved C7 63.1 mm to (82.6, 33.5), turned to 0 degrees
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Connections:
- net Net-(U1-Pad11) renamed COL2
- net Net-(U1-Pad22) renamed ROW6
- net Net-(U1-Pad26) renamed ROW7
- D2 pad 1: ROW0 -> ROW1
- D3 pad 1: ROW1 -> ROW0
- MX2 pad 1: COL1 -> COL0
- MX3 pad 1: COL0 -> COL1
- R1 pad 1: +5V -> Net-(R1-Pad1)
- U1 pad 10: Net-(U1-Pad10) -> COL3
- U1 pad 18: Net-(U1-Pad18) -> ROW1
- U1 pad 19: Net-(U1-Pad19) -> ROW2
- U1 pad 20: Net-(U1-Pad20) -> ROW3
- U1 pad 21: Net-(U1-Pad21) -> ROW4
- U1 pad 25: Net-(U1-Pad25) -> ROW5
- U1 pad 27: ROW0 -> ROW8
- U1 pad 30: ROW1 -> ROW0
- U1 pad 8: Net-(U1-Pad8) -> COL5
- U1 pad 9: Net-(U1-Pad9) -> COL4
Routing:
- net GND: track 141.6 -> 0.00 mm
- net +5V: track 97.2 -> 0.00 mm, vias 5 -> 0
- net COL1: track 51.4 -> 0.00 mm
- net ROW1: track 50.3 -> 0.00 mm
- net ROW0: track 46.4 -> 0.00 mm
- net Net-(R1-Pad2): track 33.5 -> 0.00 mm, vias 2 -> 0
- net COL0: track 32.2 -> 0.00 mm
- net Net-(R3-Pad1): track 22.1 -> 0.00 mm
- net Net-(R2-Pad1): track 21.3 -> 0.00 mm
- net Net-(C2-Pad1): track 13.0 -> 0.00 mm
- net VCC: track 11.5 -> 0.00 mm
- net Net-(C1-Pad1): track 9.98 -> 0.00 mm
- net Net-(D4-Pad2): track 6.62 -> 0.00 mm
- net Net-(D3-Pad2): track 6.62 -> 0.00 mm
- net Net-(D2-Pad2): track 6.62 -> 0.00 mm
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- removed copper zone on B.Cu, net GND
Other:
- board outline removed
- board text removed: "Hello World!"
