File: ai03-pcb-guide.sch (KiCad schematic (older format))
At the start: 24 parts, among them SW1 SW_Push, U1 ATmega32U4-AU, Y1 Crystal_GND24_Small

Commit message: lmao wtf
Parts:
- removed MX1, MX2, MX3, MX4: MX-NoLED, MX_Alps_Hybrid:MX-1U, symbol MX_Alps_Hybrid:MX-NoLED
- added D10, D11, D12, D13, D14, D15, D16, D17, D18, D19, D20, D21, D22, D23, D24, D25, D26, D27, D28, D29, D30, D31, D32, D33, D34, D35, D36, D37, D38, D39, D40, D41, D42, D43, D44, D45, D46, D47, D48, D49, D5, D50, D51, D52, D53, D54, D6, D7, D8, D9: SOD-123, random-keyboard-parts:D_SOD-123-Pretty, symbol Device:D_Small
- added MX1, MX10, MX11, MX12, MX13, MX14, MX15, MX16, MX17, MX18, MX19, MX2, MX20, MX21, MX22, MX23, MX24, MX25, MX26, MX27, MX28, MX29, MX3, MX30, MX31, MX32, MX33, MX34, MX35, MX36, MX37, MX38, MX39, MX4, MX40, MX41, MX42, MX43, MX44, MX45, MX46, MX47, MX48, MX49, MX5, MX50, MX51, MX52, MX53, MX54, MX6, MX7, MX8, MX9: MX-NoLED-MX_Alps_Hybrid, gHeavyIndustries:MX-Alps-Choc-X-1U-NoLED, symbol ai03-pcb-guide-rescue:MX-NoLED-MX_Alps_Hybrid
- C1, C2, C3, C4, C5, C6: footprint Capacitors_SMD:C_0805 -> Capacitor_SMD:C_0805_2012Metric
- C7: value 10uF -> 0.1uF; footprint Capacitors_SMD:C_0805 -> Capacitor_SMD:C_0805_2012Metric
- D1, D2, D3, D4: footprint Diodes_SMD:D_SOD-123 -> random-keyboard-parts:D_SOD-123-Pretty
- R1, R2, R3, R4: footprint Resistors_SMD:R_0805 -> Resistor_SMD:R_0805_2012Metric
- SW1: footprint random-keyboard-parts:SKQG-1155865 -> (none)
- U1: footprint Housings_QFP:TQFP-44_10x10mm_Pitch0.8mm -> Package_QFP:TQFP-44_10x10mm_P0.8mm
- USB1: footprint random-keyboard-parts:Molex-0548190589-Assembly -> random-keyboard-parts:Molex-0548190589; symbol random-keyboard-parts:Molex-0548190589 -> ai03-pcb-guide-rescue:Molex-0548190589-random-keyboard-parts
- Y1: footprint Crystals:Crystal_SMD_3225-4pin_3.2x2.5mm -> Crystal:Crystal_SMD_3225-4Pin_3.2x2.5mm
Connections:
- net labels added: COL2, COL3, COL4, COL5, COL6, COL7, COL8, ROW2, ROW3, ROW4, ROW5, ROW6, ROW7, ROW8
- wire segments 61 -> 299
Other:
- moved on the sheet: F1
